File: hardware/ti-bms.kicad_pcb (KiCad board)
At the start: 2 copper layers, 87.5 x 53 mm, 43 parts, among them J1 Conn_02x04_Odd_Even, J2 Conn_02x03_Odd_Even, J4 CAN_TERM, U1 Pico, U2 MCP2515-xST, U3 SN65HVD230, U4 TPS62160DGK, U5 MAX3485, U6 MAX3485

Commit message: more on isolation
Parts:
- added REF**: OSHW-Logo_11.4x12mm_SilkScreen, Symbol:OSHW-Logo_11.4x12mm_SilkScreen, F.Cu at (153.5, 88.5)
Other:
- net class ExtraClearance added: clearance 0.3, trace_width 0.25, via_dia 0.8, via_drill 0.4
- net class HV added: clearance 1.5, trace_width 0.25, via_dia 0.8, via_drill 0.4

Commit message: add 12v input and output, connect CAN line driver sleep pin
Parts:
- removed REF**: OSHW-Logo_11.4x12mm_SilkScreen, Symbol:OSHW-Logo_11.4x12mm_SilkScreen
- added C11: 470n, Capacitor_SMD:C_0603_1608Metric, F.Cu at (151.0, 92.5)
- added D6: 3v, Diode_SMD:D_MiniMELF, F.Cu at (148.5, 92.5)
- added Q1: NCV8402xST, Package_TO_SOT_SMD:SOT-223, F.Cu at (151.0, 81.0)
- added R13: 4k7, Resistor_SMD:R_0603_1608Metric, F.Cu at (155.0, 92.5)
- added R14: 1k5, Resistor_SMD:R_0603_1608Metric, F.Cu at (153.0, 92.5)
Connections:
- J2 pad 4: (no net) -> OUT12_1
- J2 pad 5: (no net) -> IN12_1
- U1 pad 29: (no net) -> Rs
- U1 pad 31: (no net) -> IN1
- U1 pad 32: (no net) -> OUT1
- U3 pad 8: GND -> Rs
Routing:
- net Rs: track 0.00 -> 25.7 mm
- net OUT12_1: track 0.00 -> 22.5 mm
- net IN1: track 0.00 -> 17.7 mm
- net IN12_1: track 0.00 -> 11.0 mm
- net OUT1: track 0.00 -> 9.33 mm
- net GND: track 31.7 -> 36.0 mm, vias 14 -> 20
- added copper zone on F.Cu, net OUT12_1
Other:
- board text added: "IN"
- board text added: "OUT"

Commit message: v3
Parts:
- removed the J1 at (98.5, 93.0)
- added C12: 1n 1000v, Capacitor_SMD:C_1206_3216Metric, F.Cu at (96.0, 103.5)
- added C13: 1n 1000v, Capacitor_SMD:C_1206_3216Metric, F.Cu at (96.0, 100.5)
- added C14: 100n, Capacitor_SMD:C_0603_1608Metric, F.Cu at (110.0, 98.5)
- added D7: 5v, footprints:SOD882, F.Cu at (105.5, 99.0)
- added D8: 5v, footprints:SOD882, F.Cu at (105.5, 105.0)
- added J2: Conn_01x02, Connector_Molex:Molex_Micro-Fit_3.0_43650-0200_1x02_P3.00mm_Horizontal, F.Cu at (91.5, 76.5)
- added J3: Conn_01x02, Connector_Molex:Molex_Micro-Fit_3.0_43650-0200_1x02_P3.00mm_Horizontal, F.Cu at (91.5, 90.0)
- added J4: Conn_01x02, Connector_Molex:Molex_Micro-Fit_3.0_43650-0200_1x02_P3.00mm_Horizontal, F.Cu at (91.5, 103.5)
- added L4: 22u, footprints:ACT45B-101-2P-TL003, F.Cu at (101.0, 102.0)
- added R15: 1k, Resistor_SMD:R_0603_1608Metric, F.Cu at (107.5, 103.5)
- added R16: 1k, Resistor_SMD:R_0603_1608Metric, F.Cu at (107.5, 100.5)
- added R17: 10, Resistor_SMD:R_0603_1608Metric, F.Cu at (105.0, 103.0)
- added R18: 10, Resistor_SMD:R_0603_1608Metric, F.Cu at (105.0, 101.0)
- added REF**: OSHW-Logo2_24.3x20mm_SilkScreen, Symbol:OSHW-Logo2_24.3x20mm_SilkScreen, B.Cu at (130.5, 90.0)
- added U7: MAX3485, Package_SO:SOP-8_3.9x4.9mm_P1.27mm, F.Cu at (112.5, 102.0)
- moved D3 25.0 mm to (105.5, 85.5), turned to 90 degrees
- moved R8 23.1 mm to (105.0, 87.5), turned to 0 degrees
- moved R7 20.7 mm to (105.0, 89.5), turned to 0 degrees
- moved R6 19.8 mm to (107.5, 87.0), turned to 90 degrees
- moved L3 19.0 mm to (101.0, 88.5), turned to 270 degrees
- moved D4 17.8 mm to (105.5, 91.5)
- moved R5 16.1 mm to (107.5, 90.0), turned to 90 degrees
- moved C10 15.9 mm to (110.0, 85.0), turned to 180 degrees
- moved C8 15.0 mm to (96.0, 87.0), turned to 0 degrees
- moved D2 13.1 mm to (105.5, 78.0), turned to 270 degrees
- moved U6 12.1 mm to (112.5, 88.5)
- moved C7 11.3 mm to (96.0, 90.0), turned to 0 degrees
- moved R3 11.0 mm to (105.0, 76.0), turned to 0 degrees
- moved R4 8.51 mm to (105.0, 74.0), turned to 0 degrees
- moved R1 7.78 mm to (107.5, 76.5), turned to 90 degrees
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- renumbered J2 to J1, J4 to J5
Connections:
- C5 pad 1: B1+ -> B1-
- C6 pad 1: B1- -> B1+
- C7 pad 1: B2+ -> B2-
- C8 pad 1: B2- -> B2+
- L2 pad 3: Net-(C5-Pad2) -> Net-(C6-Pad2)
- L2 pad 4: Net-(C6-Pad2) -> Net-(C5-Pad2)
- L3 pad 3: Net-(C7-Pad2) -> Net-(C8-Pad2)
- L3 pad 4: Net-(C8-Pad2) -> Net-(C7-Pad2)
- U1 pad 10: (no net) -> TXE_2
- U1 pad 11: (no net) -> RXE_2
- U1 pad 12: (no net) -> RXD_2
- U1 pad 14: TXD_2 -> TXD_3
- U1 pad 15: TXE_2 -> TXE_3
- U1 pad 16: RXE_2 -> RXE_3
- U1 pad 17: RXD_2 -> RXD_3
- U1 pad 9: (no net) -> TXD_2
Routing:
- net GND: track 36.0 -> 51.7 mm, vias 20 -> 21
- net Net-(L3-Pad1): track 14.2 -> 2.99 mm
- net TXD_3: track 0.00 -> 8.53 mm
- net Net-(L2-Pad2): track 14.2 -> 5.78 mm
- net Net-(D3-Pad1): track 13.9 -> 5.99 mm
- net Net-(D2-Pad1): track 13.9 -> 5.99 mm
- net TXE_3: track 0.00 -> 7.29 mm
- net RXE_3: track 0.00 -> 6.76 mm
- net RXD_3: track 0.00 -> 6.74 mm
- net Net-(L2-Pad1): track 9.48 -> 2.99 mm
- net Net-(C13-Pad2): track 0.00 -> 6.34 mm
- net Net-(D8-Pad1): track 0.00 -> 5.99 mm
- net Net-(D7-Pad1): track 0.00 -> 5.99 mm
- net Net-(L4-Pad2): track 0.00 -> 5.78 mm
- net Net-(D4-Pad1): track 11.2 -> 5.99 mm
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Other:
- board size 87.5 x 53 mm -> 93.5 x 53 mm
- net class HV removed
- board text added: "BATT3"
- board text added: "Daisychain BMS v3"

Commit message: dual wake inputs
Parts:
- removed Q1: NCV8402xST, Package_TO_SOT_SMD:SOT-223
- removed REF**: OSHW-Logo2_24.3x20mm_SilkScreen, Symbol:OSHW-Logo2_24.3x20mm_SilkScreen
- added C15: 1u, Capacitor_SMD:C_0603_1608Metric, F.Cu at (151.0, 83.5)
- added D9: 3v, Diode_SMD:D_MiniMELF, F.Cu at (148.5, 83.5)
- added R19: 4k7, Resistor_SMD:R_0603_1608Metric, F.Cu at (155.0, 83.5)
- added R20: 1k5, Resistor_SMD:R_0603_1608Metric, F.Cu at (153.0, 83.5)
- C11: value 470n -> 1u
- L1: footprint footprints:1227ASH100MP2 -> Inductor_SMD:L_Neosid_SMS-ME3015
- moved C11 1.00 mm to (151.0, 91.5)
- moved D6 1.00 mm to (148.5, 91.5)
- moved R13 1.00 mm to (155.0, 91.5)
- moved R14 1.00 mm to (153.0, 91.5)
- moved L1 0.25 mm to (153.0, 70.8)
Connections:
- net IN12_1 renamed WAKE1
- J1 pad 4: OUT12_1 -> WAKE2
- U1 pad 32: OUT1 -> IN2
Routing:
- net OUT12_1: track 22.5 -> 0.00 mm
- net IN2: track 0.00 -> 21.0 mm
- net WAKE2: track 0.00 -> 9.49 mm
- net OUT1: track 9.33 -> 0.00 mm
- net GND: track 51.7 -> 57.8 mm, vias 21 -> 16
- removed copper zone on F.Cu, net OUT12_1
Other:
- board text added: "WAKE"
- board text removed: "IN"
- board text removed: "OUT"

Commit message: rework inputs
Parts:
- C11, C15: value 1u -> 100n
- D6, D9: value 3v -> 3.3v
- R13, R19: value 4k7 -> 47k
- R14, R20: value 1k5 -> 4.7k
- moved C11 3.91 mm to (154.0, 89.0)
- moved R13 3.91 mm to (158.0, 89.0), turned to 270 degrees
- moved R14 3.91 mm to (156.0, 89.0)
- moved C15 3.04 mm to (154.0, 84.0)
- moved R19 3.04 mm to (158.0, 84.0), turned to 270 degrees
- moved R20 3.04 mm to (156.0, 84.0)
- moved D6 2.92 mm to (150.0, 89.0), turned to 0 degrees
- moved D9 1.58 mm to (150.0, 84.0), turned to 0 degrees
Connections:
- R13 pad 2: IN1 -> GND
- R14 pad 1: IN1 -> WAKE1
- R14 pad 2: GND -> IN1
- R19 pad 2: IN2 -> GND
- R20 pad 1: IN2 -> WAKE2
- R20 pad 2: GND -> IN2
Routing:
- net GND: track 57.8 -> 62.9 mm
- net IN2: track 21.0 -> 18.2 mm
- net WAKE1: track 10.6 -> 8.13 mm
- net IN1: track 17.2 -> 19.1 mm
- net WAKE2: track 9.49 -> 8.96 mm

Commit message: finish inputs
Parts:
- R14, R20: value 4.7k -> 5.6k

Commit message: merge v3 improvements into v2
Parts:
- removed C11, C14, C15: 100n, Capacitor_SMD:C_0603_1608Metric
- removed C12, C13: 1n 1000v, Capacitor_SMD:C_1206_3216Metric
- removed D6, D9: 3.3v, Diode_SMD:D_MiniMELF
- removed D7, D8: 5v, footprints:SOD882
- removed J3: Conn_01x02, Connector_Molex:Molex_Micro-Fit_3.0_43650-0200_1x02_P3.00mm_Horizontal
- removed the J4 at (91.5, 103.5)
- removed L4: 22u, footprints:ACT45B-101-2P-TL003
- removed R13, R19: 47k, Resistor_SMD:R_0603_1608Metric
- removed R14, R20: 5.6k, Resistor_SMD:R_0603_1608Metric
- removed R15, R16: 1k, Resistor_SMD:R_0603_1608Metric
- removed R17, R18: 10, Resistor_SMD:R_0603_1608Metric
- removed U7: MAX3485, Package_SO:SOP-8_3.9x4.9mm_P1.27mm
- added REF**: OSHW-Logo_11.4x12mm_SilkScreen, Symbol:OSHW-Logo_11.4x12mm_SilkScreen, F.Cu at (153.5, 88.5)
- J1: value Conn_02x03_Odd_Even -> Conn_02x04_Odd_Even; footprint Connector_Molex:Molex_Micro-Fit_3.0_43045-0600_2x03_P3.00mm_Horizontal -> Connector_Molex:Molex_Micro-Fit_3.0_43045-0800_2x04_P3.00mm_Horizontal
- J2: value Conn_01x02 -> Conn_02x03_Odd_Even; footprint Connector_Molex:Molex_Micro-Fit_3.0_43650-0200_1x02_P3.00mm_Horizontal -> Connector_Molex:Molex_Micro-Fit_3.0_43045-0600_2x03_P3.00mm_Horizontal
- L1: footprint Inductor_SMD:L_Neosid_SMS-ME3015 -> footprints:1227ASH100MP2
- moved J2 76.0 mm to (167.0, 85.5), turned to 270 degrees
- moved J1 68.9 mm to (98.5, 93.0), turned to 90 degrees
- moved D3 25.0 mm to (114.0, 109.0), turned to 270 degrees
- moved R8 23.1 mm to (112.0, 109.5), turned to 90 degrees
- moved R7 20.7 mm to (110.5, 109.5), turned to 90 degrees
- moved R6 19.8 mm to (113.0, 106.0), turned to 0 degrees
- moved L3 19.0 mm to (100.0, 107.5), turned to 90 degrees
- moved D4 17.8 mm to (108.5, 109.0)
- moved R5 16.1 mm to (109.5, 106.0), turned to 0 degrees
- moved C10 15.9 mm to (106.2, 100.5), turned to 90 degrees
- moved C8 15.0 mm to (101.5, 101.0), turned to 270 degrees
- moved D2 13.1 mm to (114.0, 68.0), turned to 90 degrees
- moved U6 12.1 mm to (111.0, 100.5)
- moved C7 11.3 mm to (98.5, 101.0), turned to 270 degrees
- moved R3 11.0 mm to (112.0, 67.5), turned to 270 degrees
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- renumbered J5 to J4
Connections:
- C5 pad 1: B1- -> B1+
- C6 pad 1: B1+ -> B1-
- C7 pad 1: B2- -> B2+
- C8 pad 1: B2+ -> B2-
- J1 pad 1: +12V -> B2+
- J1 pad 2: GND -> (no net)
- J1 pad 3: CANL -> (no net)
- J1 pad 4: WAKE2 -> B1-
- J1 pad 5: WAKE1 -> B2-
- J1 pad 6: CANH -> (no net)
- J2 pad 1: B1- -> +12V
- J2 pad 2: B1+ -> GND
- L2 pad 3: Net-(C6-Pad2) -> Net-(C5-Pad2)
- L2 pad 4: Net-(C5-Pad2) -> Net-(C6-Pad2)
- L3 pad 3: Net-(C8-Pad2) -> Net-(C7-Pad2)
- L3 pad 4: Net-(C7-Pad2) -> Net-(C8-Pad2)
- U1 pad 10: TXE_2 -> (no net)
- U1 pad 11: RXE_2 -> (no net)
- U1 pad 12: RXD_2 -> (no net)
- U1 pad 14: TXD_3 -> TXD_2
- U1 pad 15: TXE_3 -> TXE_2
- U1 pad 16: RXE_3 -> RXE_2
- U1 pad 17: RXD_3 -> RXD_2
- U1 pad 29: Rs -> (no net)
- U1 pad 31: IN1 -> (no net)
- U1 pad 32: IN2 -> (no net)
- U1 pad 9: TXD_2 -> (no net)
- U3 pad 8: Rs -> GND
Routing:
- net GND: track 62.9 -> 31.7 mm, vias 16 -> 14
- net Rs: track 25.7 -> 0.00 mm
- net IN1: track 19.1 -> 0.00 mm
- net IN2: track 18.2 -> 0.00 mm
- net Net-(L3-Pad1): track 2.99 -> 14.2 mm
- net WAKE2: track 8.96 -> 0.00 mm
- net TXD_3: track 8.53 -> 0.00 mm
- net Net-(L2-Pad2): track 5.78 -> 14.2 mm
- net WAKE1: track 8.13 -> 0.00 mm
- net Net-(D3-Pad1): track 5.99 -> 13.9 mm
- net Net-(D2-Pad1): track 5.99 -> 13.9 mm
- net TXE_3: track 7.29 -> 0.00 mm
- net RXE_3: track 6.76 -> 0.00 mm
- net RXD_3: track 6.74 -> 0.00 mm
- net Net-(L2-Pad1): track 2.99 -> 9.48 mm
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Other:
- board size 93.5 x 53 mm -> 87.5 x 53 mm
- net class HV added: clearance 1.5, trace_width 0.25, via_dia 0.8, via_drill 0.4
- board text removed: "BATT3"
- board text removed: "Daisychain BMS v3"
- board text removed: "WAKE"
